File: hardware/cyberbrick-breakout/kicad/cyberbrick-breakout.kicad_pcb (KiCad board)
At the start: 2 copper layers, 73 x 41 mm, 34 parts, among them J1 LX, J10 DL_LFT, J11 DL_RGT, J12 DL_DWN, J13 DR_UP, J14 DR_LFT, J15 DR_RGT, J16 DR_DWN, J17 SHL1, J18 SHL2, J19 SHR1, J2 LY, J20 SHR2, J21 START, J22 SEL, J23 HOTKEY, J24 COIN, J3 RX, J4 RY, J7 I2C, J8 PWR, J9 DL_UP, U1A ESP32-C3 top, U1B ESP32-C3 bot

Commit message: Minor changes
Parts:
- moved J7 7.46 mm to (135.0, 115.0)
- moved U1B 1.02 mm to (118.2, 118.0)
Changed lines of the file:
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@@
 		(at 178.54 127 -90)
 		(property "Reference" "J2"
-			(at 0 -2 90)
+			(at 0 -3.46 90)
 			(layer "F.SilkS")
 			(effects
@@
 		(at 148.5 118)
 		(property "Reference" "C5"
-			(at 0 -1.5 90)
+			(at 2.5 0 90)
 			(layer "F.SilkS")
 			(effects
@@
 	(footprint "Connector_PinHeader_2.54mm:PinHeader_1x04_P2.54mm_Vertical"
 		(layer "F.Cu")
-		(at 142.46 115 90)
+		(at 135 115 90)
 		(property "Reference" "J7"
 			(at 0 -3 90)
@@
 	(footprint "Connector_PinSocket_2.54mm:PinSocket_1x08_P2.54mm_Vertical"
 		(layer "B.Cu")
-		(at 118 119)
+		(at 118.22 118)
 		(property "Reference" "U1B"
 			(at -3.76 0 0)
@@
 		)
 		(pad "2" thru_hole circle
-			(at 2.54 0 90)
+			(at 2.54 0 270)
 			(size 1.6 1.6)
 			(drill 0.8)
@@
 		)
 		(pad "4" thru_hole circle
-			(at 7.62 0 90)
+			(at 7.62 0 270)
 			(size 1.6 1.6)
 			(drill 0.8)
@@
 	)
 	(gr_text "GPIO2=BOOT: no pulldown J3"
-		(at 154 115 0)
+		(at 125 125 0)
 		(layer "F.SilkS")
 		(effects
@@
 	)
 	(gr_text "CyberBrick Breakout v1.3"
-		(at 153 113 0)
+		(at 157 114 0)
 		(layer "F.SilkS")
 		(effects
@@
 		(min_thickness 0.25)
 		(filled_areas_thickness no)
-		(fill
+		(fill yes
 			(thermal_gap 0.3)
 			(thermal_bridge_width 0.3)
